Commit message: The hand as built: CAD meshes and the real finger linkages
The Fusion export in ~/Downloads/URDF_description has all 49 parts as STL but
only 2 joints (the ones defined in Fusion), so it could not replace the hand as
it is. The mechanism is recovered from the geometry instead:

- htn_description/tools/cad_to_linkage.py finds the pivots from the pin holes
  parts share (checked against the 2 exported joints: equal to 0.003 mm).
  Every finger is the same 1-DOF chain of three four-bars. It writes
  config/linkage.yaml and decimated meshes (32 MB -> 5 MB); the mannequin hand
  inside the CAD base body becomes its own 'wearer' mesh.
- htn_control/linkage.py solves the chain (circle intersections, continuation
  from the CAD pose). URDF is a tree, so each part hangs on one pivot and
  linkage_publisher publishes the 6 passive joints per finger on /joint_states.
  test_linkage.py: all loops of all fingers close to < 0.05 mm on the generated
  URDF over the whole travel.
- Contract kept: <finger>_joint (now the servo horn), 0 = open = CAD pose,
  positive closes, /hand/state 0..1. max_angle = horn angle for a 90 deg curl
  of the contact pad (72-74 deg); the linkage binds at 84-100 deg.
- Gazebo cannot close loops: sim.launch.py spawns parts:=horns (base + horns)
  while robot_state_publisher and the viewers get the full mechanism.
- Web console: backend serves /api/meshes and /api/linkage; the viewer loads
  the STLs, solves the linkage itself (TypeScript port, equal to Python to
  1e-14 rad - the commanded ghost has no passive joints on any topic), keeps
  the white/graphite look, labels on the contact pads.

Verified in an isolated sim (35 joints, TF to the pads, commands) and in the
browser (mock). NOT verified: real servos - servos.*_step calibration must be
redone, step values now mean horn angles of this linkage.

Co-Authored-By: Claude Fable 5.1 <noreply@anthropic.com>

File: application/backend/mock/hand.urdf (robot description, URDF)
Before this commit: robot htn_hand, 6 links, 5 joints
Links:
- added link index_binary; visual mesh filename=package://htn_description/meshes/index_binary.stl scale=0.001 0.001 0.001
- added link index_horn, mass 0.02; visual mesh filename=package://htn_description/meshes/index_horn.stl scale=0.001 0.001 0.001
- added link index_long; visual mesh filename=package://htn_description/meshes/index_long.stl scale=0.001 0.001 0.001
- added link index_rod; visual mesh filename=package://htn_description/meshes/index_rod.stl scale=0.001 0.001 0.001
- added link index_ternary; visual mesh filename=package://htn_description/meshes/index_ternary.stl scale=0.001 0.001 0.001
- added link index_triangle; visual mesh filename=package://htn_description/meshes/index_triangle.stl scale=0.001 0.001 0.001
- added link middle_binary; visual mesh filename=package://htn_description/meshes/middle_binary.stl scale=0.001 0.001 0.001
- added link middle_horn, mass 0.02; visual mesh filename=package://htn_description/meshes/middle_horn.stl scale=0.001 0.001 0.001
- added link middle_long; visual mesh filename=package://htn_description/meshes/middle_long.stl scale=0.001 0.001 0.001
- added link middle_rod; visual mesh filename=package://htn_description/meshes/middle_rod.stl scale=0.001 0.001 0.001
- added link middle_ternary; visual mesh filename=package://htn_description/meshes/middle_ternary.stl scale=0.001 0.001 0.001
- added link middle_triangle; visual mesh filename=package://htn_description/meshes/middle_triangle.stl scale=0.001 0.001 0.001
- added link pinky_binary; visual mesh filename=package://htn_description/meshes/pinky_binary.stl scale=0.001 0.001 0.001
- added link pinky_horn, mass 0.02; visual mesh filename=package://htn_description/meshes/pinky_horn.stl scale=0.001 0.001 0.001
- added link pinky_long; visual mesh filename=package://htn_description/meshes/pinky_long.stl scale=0.001 0.001 0.001
- added link pinky_rod; visual mesh filename=package://htn_description/meshes/pinky_rod.stl scale=0.001 0.001 0.001
- added link pinky_ternary; visual mesh filename=package://htn_description/meshes/pinky_ternary.stl scale=0.001 0.001 0.001
- added link pinky_triangle; visual mesh filename=package://htn_description/meshes/pinky_triangle.stl scale=0.001 0.001 0.001
- added link ring_binary; visual mesh filename=package://htn_description/meshes/ring_binary.stl scale=0.001 0.001 0.001
- added link ring_horn, mass 0.02; visual mesh filename=package://htn_description/meshes/ring_horn.stl scale=0.001 0.001 0.001
- added link ring_long; visual mesh filename=package://htn_description/meshes/ring_long.stl scale=0.001 0.001 0.001
- added link ring_rod; visual mesh filename=package://htn_description/meshes/ring_rod.stl scale=0.001 0.001 0.001
- added link ring_ternary; visual mesh filename=package://htn_description/meshes/ring_ternary.stl scale=0.001 0.001 0.001
- added link ring_triangle; visual mesh filename=package://htn_description/meshes/ring_triangle.stl scale=0.001 0.001 0.001
- added link thumb_binary; visual mesh filename=package://htn_description/meshes/thumb_binary.stl scale=0.001 0.001 0.001
- added link thumb_horn, mass 0.02; visual mesh filename=package://htn_description/meshes/thumb_horn.stl scale=0.001 0.001 0.001
- added link thumb_long; visual mesh filename=package://htn_description/meshes/thumb_long.stl scale=0.001 0.001 0.001
- added link thumb_rod; visual mesh filename=package://htn_description/meshes/thumb_rod.stl scale=0.001 0.001 0.001
- added link thumb_ternary; visual mesh filename=package://htn_description/meshes/thumb_ternary.stl scale=0.001 0.001 0.001
- added link thumb_triangle; visual mesh filename=package://htn_description/meshes/thumb_triangle.stl scale=0.001 0.001 0.001
- link base_link: mass 0.15 -> 0.63; geometry visual mesh filename=package://htn_description/meshes/base.stl scale=0.001 0.001 0.001; visual mesh filename=package://htn_description/meshes/wearer.stl scale=0.001 0.001 0.001
- link index_finger: mass 0.02 -> None; geometry visual mesh filename=package://htn_description/meshes/index_adapter.stl scale=0.001 0.001 0.001; visual mesh filename=package://htn_description/meshes/index_contact.stl scale=0.001 0.001 0.001
- link middle_finger: mass 0.02 -> None; geometry visual mesh filename=package://htn_description/meshes/middle_adapter.stl scale=0.001 0.001 0.001; visual mesh filename=package://htn_description/meshes/middle_contact.stl scale=0.001 0.001 0.001
- link pinky_finger: mass 0.02 -> None; geometry visual mesh filename=package://htn_description/meshes/pinky_adapter.stl scale=0.001 0.001 0.001; visual mesh filename=package://htn_description/meshes/pinky_contact.stl scale=0.001 0.001 0.001
- link ring_finger: mass 0.02 -> None; geometry visual mesh filename=package://htn_description/meshes/ring_adapter.stl scale=0.001 0.001 0.001; visual mesh filename=package://htn_description/meshes/ring_contact.stl scale=0.001 0.001 0.001
- link thumb_finger: mass 0.02 -> None; geometry visual mesh filename=package://htn_description/meshes/thumb_adapter.stl scale=0.001 0.001 0.001; visual mesh filename=package://htn_description/meshes/thumb_contact.stl scale=0.001 0.001 0.001
Joints:
- added joint index_adapter_joint: type continuous, parent index_ternary, child index_finger, origin xyz=0.0 0.020239999999999994 -0.04297, axis 1 0 0
- added joint index_binary_joint: type continuous, parent index_long, child index_binary, origin xyz=0.0 0.0 0.0475, axis 1 0 0
- added joint index_long_joint: type continuous, parent base_link, child index_long, origin xyz=0.078 0.05771 0.02705, axis 1 0 0
- added joint index_rod_joint: type continuous, parent index_horn, child index_rod, origin xyz=0.0 -0.007449999999999999 0.01507, axis 1 0 0
- added joint index_ternary_joint: type continuous, parent index_triangle, child index_ternary, origin xyz=0.0 -9.99999999999801e-06 0.028999999999999995, axis 1 0 0
- added joint index_triangle_joint: type continuous, parent base_link, child index_triangle, origin xyz=0.078 0.04962 0.04424, axis 1 0 0
- added joint middle_adapter_joint: type continuous, parent middle_ternary, child middle_finger, origin xyz=0.0 0.020239999999999994 -0.04297, axis 1 0 0
- added joint middle_binary_joint: type continuous, parent middle_long, child middle_binary, origin xyz=0.0 0.0 0.0475, axis 1 0 0
- added joint middle_long_joint: type continuous, parent base_link, child middle_long, origin xyz=0.055 0.05771 0.02705, axis 1 0 0
- added joint middle_rod_joint: type continuous, parent middle_horn, child middle_rod, origin xyz=0.0 -0.00745 0.01507, axis 1 0 0
- added joint middle_ternary_joint: type continuous, parent middle_triangle, child middle_ternary, origin xyz=0.0 -9.99999999999801e-06 0.028999999999999995, axis 1 0 0
- added joint middle_triangle_joint: type continuous, parent base_link, child middle_triangle, origin xyz=0.055 0.04962 0.04424, axis 1 0 0
- added joint pinky_adapter_joint: type continuous, parent pinky_ternary, child pinky_finger, origin xyz=0.0 0.020239999999999994 -0.04297, axis 1 0 0
- added joint pinky_binary_joint: type continuous, parent pinky_long, child pinky_binary, origin xyz=0.0 0.0 0.0475, axis 1 0 0
- added joint pinky_long_joint: type continuous, parent base_link, child pinky_long, origin xyz=0.01 0.05771 0.02705, axis 1 0 0
- added joint pinky_rod_joint: type continuous, parent pinky_horn, child pinky_rod, origin xyz=0.0 -0.007449999999999999 0.01507, axis 1 0 0
- added joint pinky_ternary_joint: type continuous, parent pinky_triangle, child pinky_ternary, origin xyz=0.0 -9.99999999999801e-06 0.028999999999999995, axis 1 0 0
- added joint pinky_triangle_joint: type continuous, parent base_link, child pinky_triangle, origin xyz=0.01 0.04962 0.04424, axis 1 0 0
- added joint ring_adapter_joint: type continuous, parent ring_ternary, child ring_finger, origin xyz=0.0 0.020239999999999994 -0.04297, axis 1 0 0
- added joint ring_binary_joint: type continuous, parent ring_long, child ring_binary, origin xyz=0.0 0.0 0.0475, axis 1 0 0
- added joint ring_long_joint: type continuous, parent base_link, child ring_long, origin xyz=0.033 0.05771 0.02705, axis 1 0 0
- added joint ring_rod_joint: type continuous, parent ring_horn, child ring_rod, origin xyz=0.0 -0.00745 0.01507, axis 1 0 0
- added joint ring_ternary_joint: type continuous, parent ring_triangle, child ring_ternary, origin xyz=0.0 -9.99999999999801e-06 0.028999999999999995, axis 1 0 0
- added joint ring_triangle_joint: type continuous, parent base_link, child ring_triangle, origin xyz=0.033 0.04962 0.04424, axis 1 0 0
- added joint thumb_adapter_joint: type continuous, parent thumb_ternary, child thumb_finger, origin xyz=-0.03346 0.03372 0.0, axis 0 0 1
- added joint thumb_binary_joint: type continuous, parent thumb_long, child thumb_binary, origin xyz=0.04464 -0.01625 0.0, axis 0 0 1
- added joint thumb_long_joint: type continuous, parent base_link, child thumb_long, origin xyz=0.12036 0.008369999999999999 -0.026760000000000003, axis 0 0 1
- added joint thumb_rod_joint: type continuous, parent thumb_horn, child thumb_rod, origin xyz=0.011609999999999999 -0.012160000000000004 0.0, axis 0 0 1
- added joint thumb_ternary_joint: type continuous, parent thumb_triangle, child thumb_ternary, origin xyz=0.02725 -0.00993 0.0, axis 0 0 1
- added joint thumb_triangle_joint: type continuous, parent base_link, child thumb_triangle, origin xyz=0.13375 -0.00511 -0.026760000000000003, axis 0 0 1
- joint index_joint: axis 0 1 0 -> -1 0 0; child index_finger -> index_horn; limit lower=0.0 upper=1.57 effort=1.0 velocity=3.0 -> lower=0.0 upper=1.2828 effort=1.0 velocity=3.0; origin xyz=0.03 -0.033 0.0 rpy=-0.0 0.0 -0.0 -> xyz=0.078 0.03188 0.04446
- joint middle_joint: axis 0 1 0 -> -1 0 0; child middle_finger -> middle_horn; limit lower=0.0 upper=1.57 effort=1.0 velocity=3.0 -> lower=0.0 upper=1.2523 effort=1.0 velocity=3.0; origin xyz=0.03 -0.011 0.0 rpy=-0.0 0.0 -0.0 -> xyz=0.055 0.00588 0.04446
- joint pinky_joint: axis 0 1 0 -> -1 0 0; child pinky_finger -> pinky_horn; limit lower=0.0 upper=1.57 effort=1.0 velocity=3.0 -> lower=0.0 upper=1.2828 effort=1.0 velocity=3.0; origin xyz=0.03 0.033 0.0 rpy=-0.0 0.0 -0.0 -> xyz=0.01 0.03188 0.04446
- joint ring_joint: axis 0 1 0 -> -1 0 0; child ring_finger -> ring_horn; limit lower=0.0 upper=1.57 effort=1.0 velocity=3.0 -> lower=0.0 upper=1.2523 effort=1.0 velocity=3.0; origin xyz=0.03 0.011 0.0 rpy=-0.0 0.0 -0.0 -> xyz=0.033 0.00588 0.04446
- joint thumb_joint: axis 0 1 0 -> 0 0 1; child thumb_finger -> thumb_horn; limit lower=0.0 upper=1.57 effort=1.0 velocity=3.0 -> lower=0.0 upper=1.2828 effort=1.0 velocity=3.0; origin xyz=-0.02 -0.055 0.0 rpy=-0.0 0.0 -1.5708 -> xyz=0.12789 -0.02186 -0.026760000000000003
